File: pcb/usb_c.sch (KiCad schematic (older format))
At the start: 33 parts, among them J401 USB_C_Receptacle_USB2.0, M401 MPMOS, M402 MPMOS, U401 STUSB1602, U402 L7985

Commit message: [PCB] minor changes
Parts:
- removed C401, C402, C403: 1u, symbol Device:C_Small
- removed R401, R403, R405, R406, R407, R409, R410, R412: 10k, symbol Device:R_Small
- removed R402, R404, R408: 1k, symbol Device:R_Small
- added C? (x3): 1u, Capacitor_SMD:C_0603_1608Metric, symbol Device:C_Small
- added JP?: SolderJumper_3_Open, symbol Jumper:SolderJumper_3_Open
- added R? (x7): 10k, symbol Device:R_Small
- added R? (x3): 1k, symbol Device:R_Small
- C404, C405, C406, C407, C408, C409: footprint (none) -> Capacitor_SMD:C_0603_1608Metric
- D401: footprint (none) -> Diode_SMD:D_0201_0603Metric
- J401: footprint (none) -> Connector_USB:USB_C_Receptacle_HRO_TYPE-C-31-M-12
Connections:
- net +3V3: now also U401.22 (VSYS), JP?.1 (A), R?.2, R?.2, R?.2, R?.2, R?.2, R?.2
- net ALERT#: now also R?.1
- net GND: now also C?.1, C?.1, C?.2, JP?.3 (B), R?.1, R?.1
- net MOSI: now also R?.1
- net NSS: now also R?.1
- net RESET: now also R?.2
- net SCL: now also R?.1
- net SCLK: now also R?.1
- net SDA: now also R?.1
- net TX_EN: now also R?.2
- net at U401.23 (VReg_2V7): now also C?.1
- net at U401.21 (VReg_1V2): now also C?.2
- net at J401.A4 (VBUS), J401.A9 (VBUS), J401.B4 (VBUS)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: now also C?.2
- net at U401.19 (VBUS_EN_SNK): now also R?.1
- net at M401.3 (S), M401.4 (B), M402.3 (S)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: now also R?.2
- net at M401.2 (G), M402.2 (G): now also R?.1, R?.2
- net USB_D+: now reaches J401.A6 (D+), J401.B6 (D+)
- net USB_D-: now reaches J401.A7 (D-), J401.B7 (D-)
- net AB_SIDE: no longer names the net of U401.17 (AB_SIDE)
- net ADDR0: no longer names the net of U401.13 (ADDR0)
- net ADDR0: now also JP?.2 (C)
- no-connect marks 4 -> 5
Other:
- moved on the sheet: C404, C406, C407, R411

Commit message: [PCB] corrections composants
Parts:
- added C? (x2): 1u, Capacitor_SMD:C_0603_1608Metric, symbol Device:C_Small
- J401: symbol Connector:USB_C_Receptacle_USB2.0 -> usb_alim-rescue:USB_C_Receptacle_USB2.0-Connector
Connections:
- net +3V3: now also C?.1
- net GND: now also C?.2
- net at M401.3 (S), M401.4 (B), M402.3 (S)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: now also C?.2
- net at M401.2 (G), M402.2 (G), R?.1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: now also C?.1
Other:
- note added: "Dans le DOC ils mettent 10k,\ntrès honnetement je sais pas\nsi ça change grand chose\n"
- note added: "Il y a des jumpers dans UM2191,\nentre CCX et CCXDB,\ntu sais pourquoi ?"
- note added: "Pour SCLK ils mettent 2.2k dans le doc UM2191,\nà voir dans la datasheet"
- moved on the sheet: R?
Changed lines of the file:
@@
 	6000 2650 6000 2600
 Wire Wire Line
-	6000 2600 5500 2600
-Wire Wire Line
 	5500 2600 5500 2550
 Wire Wire Line
-	6000 2600 6300 2600
+	6000 2600 6050 2600
 Wire Wire Line
 	6300 2600 6300 2550
 Connection ~ 6000 2600
-Wire Wire Line
-	6000 2550 6000 2600
-Wire Wire Line
-	6000 2250 6100 2250
-Wire Wire Line
-	6000 2250 6000 2350
-Wire Wire Line
-	5700 2250 5800 2250
-Connection ~ 6000 2250
 Connection ~ 7500 1250
 Wire Wire Line
@@
 Wire Wire Line
 	6000 2850 6000 2950
-Connection ~ 5800 2250
-Wire Wire Line
-	5800 2250 6000 2250
-Wire Wire Line
-	5800 2250 5800 2950
 $Comp
 L pspice:MPMOS M401
@@
 	4900 3250 4900 3550
 $Comp
-L Connector:USB_C_Receptacle_USB2.0 J401
+L usb_alim-rescue:USB_C_Receptacle_USB2.0-Connector J401
 U 1 1 607E779C
 P 3550 3650
+AR Path="/607E779C" Ref="J401"  Part="1"
+AR Path="/6071A9E5/607E779C" Ref="J401"  Part="1"
 F 0 "J401" H 3657 4517 50  0000 C CNN
 F 1 "USB_C_Receptacle_USB2.0" H 3657 4426 50  0000 C CNN
@@
 L Device:R_Small R?
 U 1 1 60680349
-P 6000 2450
-F 0 "R?" V 5950 2450 39  0000 C BNN
-F 1 "10k" V 6050 2450 39  0000 C TNN
-F 2 "" H 6000 2450 50  0001 C CNN
-F 3 "~" H 6000 2450 50  0001 C CNN
-	1    6000 2450
+P 6050 2450
+F 0 "R?" V 6000 2450 39  0000 C BNN
+F 1 "10k" V 6100 2450 39  0000 C TNN
+F 2 "" H 6050 2450 50  0001 C CNN
+F 3 "~" H 6050 2450 50  0001 C CNN
+	1    6050 2450
 	1    0    0    1
 $EndComp
@@
 	6900 4650 7150 4650
 Wire Wire Line
-	6300 2950 6650 2950
+	6300 2950 6450 2950
 Wire Wire Line
 	6650 2950 6650 2600
@@
 	4200 3750 4250 3750
 Connection ~ 4200 3750
+$Comp
+L Device:C_Small C?
+U 1 1 6077C8BA
+P 6450 2850
+F 0 "C?" V 6350 2850 39  0000 C CNN
+F 1 "1u" V 6550 2850 39  0000 C CNN
+F 2 "Capacitor_SMD:C_0603_1608Metric" H 6450 2850 50  0001 C CNN
+F 3 "~" H 6450 2850 50  0001 C CNN
+	1    6450 2850
+	1    0    0    1
+$EndComp
+Connection ~ 6450 2950
+Wire Wire Line
+	6450 2950 6650 2950
+$Comp
+L power:GND #PWR?
+U 1 1 6077CF57
+P 6450 2750
+F 0 "#PWR?" H 6450 2500 50  0001 C CNN
+F 1 "GND" H 6450 2650 39  0000 C TNN
+F 2 "" H 6450 2750 50  0001 C CNN
+F 3 "" H 6450 2750 50  0001 C CNN
+	1    6450 2750
+	-1   0    0    1
+$EndComp
+Text Notes 8800 3500 0    50   ~ 0
+Pour SCLK ils mettent 2.2k dans le doc UM2191,\nà voir dans la datasheet
+Text Notes 6850 4800 0    50   ~ 0
+Dans le DOC ils mettent 10k,\ntrès honnetement je sais pas\nsi ça change grand chose\n
+Text Notes 4200 3500 0    50   ~ 0
+Il y a des jumpers dans UM2191,\nentre CCX et CCXDB,\ntu sais pourquoi ?
+$Comp
+L Device:C_Small C?
+U 1 1 60783CC0
+P 5800 2450
+F 0 "C?" V 5700 2450 39  0000 C CNN
+F 1 "1u" V 5900 2450 39  0000 C CNN
+F 2 "Capacitor_SMD:C_0603_1608Metric" H 5800 2450 50  0001 C CNN
+F 3 "~" H 5800 2450 50  0001 C CNN
+	1    5800 2450
+	1    0    0    1
+$EndComp
+Wire Wire Line
+	5700 2250 5750 2250
+Wire Wire Line
+	5800 2950 5800 2800
+Wire Wire Line
+	5800 2800 5750 2800
+Wire Wire Line
+	5750 2800 5750 2250
+Connection ~ 5750 2250
+Wire Wire Line
+	5750 2250 5800 2250
+Wire Wire Line
+	5500 2600 5800 2600
+Wire Wire Line
+	5800 2550 5800 2600
+Connection ~ 5800 2600
+Wire Wire Line
+	5800 2600 6000 2600
+Wire Wire Line
+	5800 2350 5800 2250
+Connection ~ 5800 2250
+Wire Wire Line
+	5800 2250 6050 2250
+Wire Wire Line
+	6050 2550 6050 2600
+Connection ~ 6050 2600
+Wire Wire Line
+	6050 2600 6300 2600
+Wire Wire Line
+	6050 2350 6050 2250
+Connection ~ 6050 2250
+Wire Wire Line
+	6050 2250 6100 2250
 $EndSCHEMATC
